Commit message: new lidar model

File: Diff_Robot_model/diff_drive_bot_with_lidar2/urdf/diff_drive_bot_with_lidar.urdf (robot description, URDF)
Before this commit: robot diff_drive_bot_with_lidar, 4 links, 3 joints
Links:
- removed link lidar_link
- link right_link: mass 0.215827415301619 -> 0.21583
Joints:
- removed joint lidar_joint

Commit message: lidar rotor seperated

File: Diff_Robot_model/diff_drive_bot_with_lidar2/urdf/diff_drive_bot_with_lidar.urdf (robot description, URDF)
Before this commit: robot diff_drive_bot_with_lidar, 5 links, 4 joints
Links:
- removed link lidar_base_link
- removed link lidar_rot_link
- added link lidar_link, mass 0; collision mesh filename=package://diff_drive_bot_with_lidar/meshes/lidar_link.STL; visual mesh filename=package://diff_drive_bot_with_lidar/meshes/lidar_link.STL
- link base_link: mass 2.77638109182328 -> 2.7764
- link left_link: mass 0.215827415301619 -> 0.21583
Joints:
- removed joint lidar_base_joint
- removed joint lidar_rot_joint
- added joint lidar_joint: type fixed, parent base_link, child lidar_link, origin xyz=-0.0028128 -0.004107 0.1281 rpy=0 0 -0.053034, axis 0 0 0
- joint left_wheel: origin xyz=-0.138666895478107 0.139916380652366 -0.042 rpy=0 0 0 -> xyz=-0.13867 0.13992 -0.042 rpy=0 0 0
