Commit message: replaced old lidar model

File: diff_driver_ros_tut/src/diff_drive_bot_with_lidar/urdf/diff_drive_bot_with_lidar.urdf (robot description, URDF)
Before this commit: robot diff_drive_bot_with_lidar, 3 links, 2 joints
Links:
- added link lidar_link, mass 0; collision mesh filename=package://diff_drive_bot_with_lidar/meshes/lidar_link.STL; visual mesh filename=package://diff_drive_bot_with_lidar/meshes/lidar_link.STL
- link right_link: mass 0.21583 -> 0.215827415301619
Joints:
- added joint lidar_joint: type fixed, parent base_link, child lidar_link, origin xyz=-0.0028128 -0.004107 0.1281 rpy=0 0 -0.053034, axis 0 0 0
- joint left_wheel: axis 0 1 0 -> 0 -1 0
- joint right_wheel: axis 0 1 0 -> 0 -1 0

Commit message: code for lidar

File: diff_driver_ros_tut/src/diff_drive_bot_with_lidar/urdf/diff_drive_bot_with_lidar.urdf (robot description, URDF)
Before this commit: robot diff_drive_bot_with_lidar, 5 links, 4 joints
Joints:
- joint left_wheel: axis 0 -1 0 -> 0 1 0
- joint right_wheel: axis 0 -1 0 -> 0 1 0
