Commit message: replaced again

File: Diff_Robot_model/diff_drive_bot_with_lidar/urdf/diff_drive_bot_with_lidar.urdf (robot description, URDF)
Before this commit: robot diff_drive_bot_with_lidar, 5 links, 4 joints
Joints:
- joint lidar_base_joint: origin xyz=-0.010334 -0.0035917 0.1 rpy=0 0 -0.053034 -> xyz=-0.0103343023948472 -0.00359165195948655 0.1 rpy=0 0 -0.0530343084887313
- joint lidar_rot_joint: origin xyz=-0.0027573 -0.0040961 0.1281 rpy=0 0 -0.053034 -> xyz=-0.00275728157019983 -0.00409611162826763 0.1281 rpy=0 0 -0.0530343084887313
- joint right_wheel: origin xyz=-0.13867 -0.14208 -0.042 rpy=0 0 0 -> xyz=-0.138666895478107 -0.142083619347635 -0.042 rpy=0 0 0

Commit message: base_link changes

File: Diff_Robot_model/diff_drive_bot_with_lidar/urdf/diff_drive_bot_with_lidar.urdf (robot description, URDF)
Before this commit: robot diff_drive_bot_with_lidar, 5 links, 4 joints
Joints:
- joint left_wheel: origin xyz=-0.138666895478107 0.139916380652366 -0.042 rpy=0 0 0 -> xyz=0 0.141 -0.042 rpy=0 0 0
- joint lidar_base_joint: origin xyz=-0.0103343023948472 -0.00359165195948655 0.1 rpy=0 0 -0.0530343084887313 -> xyz=0.12833 -0.002508 0.1 rpy=0 0 -0.053034
- joint lidar_rot_joint: origin xyz=-0.00275728157019983 -0.00409611162826763 0.1281 rpy=0 0 -0.0530343084887313 -> xyz=0.13591 -0.0030125 0.1281 rpy=0 0 -0.053034
- joint right_wheel: origin xyz=-0.138666895478107 -0.142083619347635 -0.042 rpy=0 0 0 -> xyz=0 -0.141 -0.042 rpy=0 0 0

Commit message: replaced

File: Diff_Robot_model/diff_drive_bot_with_lidar/urdf/diff_drive_bot_with_lidar.urdf (robot description, URDF)
Before this commit: robot diff_drive_bot_with_lidar, 4 links, 3 joints
Links:
- removed link lidar_link
- added link lidar_base_link, mass 1.33982083389145; collision mesh filename=package://diff_drive_bot_with_lidar/meshes/lidar_base_link.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; visual mesh filename=package://diff_drive_bot_with_lidar/meshes/lidar_base_link.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
- added link lidar_rot_link, mass 0.838797463919277; collision mesh filename=package://diff_drive_bot_with_lidar/meshes/lidar_rot_link.S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; visual mesh filename=package://diff_drive_bot_with_lidar/meshes/lidar_rot_link.S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
- link base_link: mass 2.7764 -> 2.77638109182328
- link left_link: mass 0.21583 -> 0.215827415301619
Joints:
- removed joint lidar_joint
- added joint lidar_base_joint: type fixed, parent base_link, child lidar_base_link, origin xyz=0.12833259308326 -0.00250803261185217 0.1 rpy=0 0 -0.0530343084887313, axis 0 0 0
- added joint lidar_rot_joint: type continuous, parent base_link, child lidar_rot_link, origin xyz=0.135909613907908 -0.00301249228063324 0.1281 rpy=0 0 -0.0530343084887313, axis 0 0 1, limit effort=1 velocity=1
- joint left_wheel: origin xyz=-0.13867 0.13992 -0.042 rpy=0 0 0 -> xyz=0 0.141 -0.042 rpy=0 0 0
- joint right_wheel: origin xyz=-0.13867 -0.14208 -0.042 rpy=0 0 0 -> xyz=0 -0.141 -0.042 rpy=0 0 0

File: diff_driver_ros_tut/src/diff_drive_bot_with_lidar/urdf/diff_drive_bot_with_lidar.urdf (robot description, URDF)
Before this commit: robot diff_drive_bot_with_lidar, 5 links, 4 joints
Joints:
- joint lidar_base_joint: origin xyz=0.12833 -0.002508 0.1 rpy=0 0 -0.053034 -> xyz=0.12833259308326 -0.00250803261185217 0.1 rpy=0 0 -0.0530343084887313
- joint lidar_rot_joint: origin xyz=0.13591 -0.0030125 0.1281 rpy=0 0 -0.053034 -> xyz=0.135909613907908 -0.00301249228063324 0.1281 rpy=0 0 -0.0530343084887313
